Commit message: resolve

File: HYUSPA/hyuspa_description/urdf/right_sim.xacro (robot description, xacro)
@@ -9,4 +9,10 @@
   <joint name="world_base" type="fixed">
     <parent link="world"/>
+    <child link="Arm_Link_base"/>
+    <origin xyz="0 0 0" rpy="0 0 0"/>
+  </joint>
+  <link name="Arm_Link_base"/>
+  <joint name="Arm_Joint_base_joint" type="fixed">
+    <parent link="Arm_Link_base"/>
     <child link="Arm_Link_00"/>
     <origin xyz="0 0 0" rpy="0 0 0"/>
