Commit message: Controller

File: HYUSPA/hyuspa_description/urdf/links_joints.xacro (robot description, xacro)
@@ -98,10 +98,4 @@
         <inertia ixx="${ixx}" ixy="${ixy}" ixz="${ixz}" iyy="${iyy}" iyz="${iyz}" izz="${izz}" />
       </inertial>
-      <collision>
-        <origin rpy="${colvis_rpy}" xyz="${colvis_xyz}" />
-        <geometry>
-          <mesh filename="${meshfile}" scale="${meshscale}"/>
-        </geometry>
-      </collision>
       <visual>
         <origin rpy="${colvis_rpy}" xyz="${colvis_xyz}" />
@@ -113,4 +107,10 @@
     </link>
   </xacro:macro>
+<!--  <collision>
+    <origin rpy="${colvis_rpy}" xyz="${colvis_xyz}" />
+    <geometry>
+      <mesh filename="${meshfile}" scale="${meshscale}"/>
+    </geometry>
+  </collision>-->
 </robot>
 <!--

File: HYUSPA/hyuspa_description/urdf/right_sim.xacro (robot description, xacro)
@@ -30,6 +30,6 @@
            axis_xyz="0 1 0"
            origin_rpy="0 0 3.1416" origin_xyz="0 -0.2305 1.567"
-           parent="Arm_Link_00" child="Arm_Link_01" damping="0.7" friction="1.0"
-           limit_e="1000" limit_l="-1.11" limit_u="3.09" limit_v="2.4" />
+           parent="Arm_Link_00" child="Arm_Link_01" damping="0.0" friction="0.7"
+           limit_e="50" limit_l="-1.11" limit_u="3.09" limit_v="2.4" />
   <m_link_mesh name="${link_01_name}"
               origin_rpy="0 0 0" origin_xyz="0.00084 0.033665 -0.00002"
@@ -44,6 +44,6 @@
            axis_xyz="1 0 0"
            origin_rpy="0 0 0" origin_xyz="0 0.05 0"
-           parent="Arm_Link_01" child="Arm_Link_02" damping="0.7" friction="1.0"
-           limit_e="1000" limit_l="-1.57" limit_u="1.57" limit_v="2.4" />
+           parent="Arm_Link_01" child="Arm_Link_02" damping="0.0" friction="0.7"
+           limit_e="50" limit_l="-1.9" limit_u="1.57" limit_v="2.4" />
   <m_link_mesh name="${link_02_name}"
               origin_rpy="0 0 0" origin_xyz="0.00366 0.10318 0.00003"
@@ -58,6 +58,6 @@
            axis_xyz="0 1 0"
            origin_rpy="0 0 0" origin_xyz="0 0.18525 0"
-           parent="Arm_Link_02" child="Arm_Link_03" damping="0.7" friction="1.0"
-           limit_e="1000" limit_l="-1.34" limit_u="1.09" limit_v="2.4" />
+           parent="Arm_Link_02" child="Arm_Link_03" damping="0.0" friction="0.7"
+           limit_e="50" limit_l="-1.34" limit_u="1.09" limit_v="2.4" />
   <m_link_mesh name="${link_03_name}"
               origin_rpy="0 0 0" origin_xyz="0.0030362 0.06202 0.00069786"
@@ -72,6 +72,6 @@
            axis_xyz="0 0 1"
            origin_rpy="0 0 0" origin_xyz="0 0.1168 0"
-           parent="Arm_Link_03" child="Arm_Link_04" damping="0.7" friction="1.0"
-           limit_e="1000" limit_l="-0.156" limit_u="2.48" limit_v="2.4" />
+           parent="Arm_Link_03" child="Arm_Link_04" damping="0.0" friction="0.7"
+           limit_e="50" limit_l="-0.156" limit_u="2.48" limit_v="2.4" />
   <m_link_mesh name="${link_04_name}"
               origin_rpy="0 0 0" origin_xyz="0.00004 0.041284 -0.00463"
@@ -86,6 +86,6 @@
            axis_xyz="0 1 0"
            origin_rpy="0 0 0" origin_xyz="0 0.1274 0"
-           parent="Arm_Link_04" child="Arm_Link_05" damping="0.7" friction="1.0"
-           limit_e="1000" limit_l="-1.41" limit_u="1.392" limit_v="2.4" />
+           parent="Arm_Link_04" child="Arm_Link_05" damping="0.0" friction="0.7"
+           limit_e="50" limit_l="-1.41" limit_u="1.392" limit_v="2.4" />
   <m_link_mesh name="${link_05_name}"
               origin_rpy="0 0 0" origin_xyz="-0.00229 0.13004 0.00324"
@@ -98,4 +98,16 @@
               meshscale="1 1 1" />
   <!-- END - Robot description -->
+  	<gazebo>
+		<plugin name="p3d_base_controller" filename="libgazebo_ros_p3d.so">
+			<alwaysOn>true</alwaysOn>
+			<updateRate>1000.0</updateRate>
+			<bodyName>Arm_Link_05</bodyName>
+			<topicName>ground_truth/state</topicName>
+			<gaussianNoise>0</gaussianNoise>
+			<frameName>world</frameName>
+			<xyzOffsets>0 0 0</xyzOffsets>
+			<rpyOffsets>0 0 0</rpyOffsets>
+		</plugin>
+	</gazebo>
   <gazebo>
     <plugin name="gazebo_ros_control" filename="libgazebo_ros_control.so">
